File: kicad/ISLKey.kicad_sch (KiCad schematic)
At the start: 43 parts, among them J10 5-60V AC/DC IN, J11 12V OUT (lock/aux), J13 TTGO batt pads, J15 DCDC ON link (Ctrl-+Vin), J3 Exit btn, J4 Door contact, J5 Tamper, J6 LOCK COM/NO/NC, J7 AUX COM/NO/NC, J8 Fire volt-free, J9 Fire link COM-Fire, K1 SRD-05VDC-SL-C, K2 SRD-05VDC-SL-C, M1 TTGO T-Display, Q1 PN2222A, Q2 PN2222A, U1 PC817, U3 TMR10-2412WIR, U4 TSR-1-2450, U5 DS3231M

Commit message: Release v1.0.0 — ISLKey 1-MDC
Freeze the full-featured controller as v1.0.0 "1-MDC": TTGO carrier, 4 inputs
(exit/door/fire/tamper), dual relays w/ status LEDs, monitored fire link,
DS3231 RTC, single 18650 backup, wide-input isolated PSU (TMR10 -> TSR buck),
SMD passives, perimeter terminals, fully routed (148x128mm), turnkey BOM +
PCBWay package.

Co-Authored-By: Claude Opus 4.8 <noreply@anthropic.com>
Claude-Session: https://claude.ai/code/session_01WaJbCVpNNC7xF4fkqWpjpA
Other:
- title: ISLKey TTGO Carrier Board -> ISLKey 1-MDC
Changed lines of the file:
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@@
   (generator "islkey_gen") (generator_version "10.0")
   (paper "A3")
-  (title_block (title "ISLKey TTGO Carrier Board") (company "ISL Technologies") (rev "2.0.0")
-    (comment 1 "Inputs, dual onboard relays w/ status LEDs, monitored fire link, backup-power passthrough"))
+  (title_block (title "ISLKey 1-MDC") (company "ISL Technologies") (rev "1.0.0")
+    (comment 1 "1-MDC: TTGO controller - 4 inputs, dual relays, monitored fire link, RTC, wide-input isolated PSU"))
   (wire (pts (xy 63.5 97.79) (xy 67.31 97.79)) (stroke (width 0) (type default)))
   (global_label "+5V" (shape bidirectional) (at 67.31 97.79 0) (fields_autoplaced yes)
